File: ESC_BLDC.kicad_pcb (KiCad board)
At the start: 4 copper layers, 70 x 90 mm, 95 parts, among them J1 Conn_01x06_Pin, J2 Conn_01x04_Pin, U4 LM339, U5 AP1509-50SG-13, U6 MCP6002-xP, U7 MCP6002-xP, U8 MCP6002-xP

Commit message: ordenado por funcion
Parts:
- DBUCK1: footprint Diode_SMD:D_1206_3216Metric_Pad1.42x1.75mm_HandSolder -> Diode_THT:D_DO-34_SOD68_P7.62mm_Horizontal
- moved CdesA1 138.6 mm to (144.0, 187.2)
- moved CdesB1 138.6 mm to (144.0, 190.5)
- moved CdesC1 138.6 mm to (144.0, 193.9)
- moved U5 136.4 mm to (107.0, 191.3)
- moved RN2 132.6 mm to (151.9, 183.7)
- moved RN3 132.6 mm to (151.9, 187.0)
- moved RN5 132.6 mm to (151.9, 193.6)
- moved RN1 132.6 mm to (151.9, 180.4)
- moved RN4 132.6 mm to (151.9, 190.3)
- moved CDESBEMF1 126.4 mm to (144.1, 176.7)
- moved CDESBEMF2 126.4 mm to (144.1, 180.0)
- moved CDESBEMF3 126.4 mm to (144.1, 183.4)
- moved CADES1 125.5 mm to (20.0, 188.8)
- moved CdesN1 124.8 mm to (151.9, 177.0)
- moved U6 120.5 mm to (130.5, 167.3)
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Connections:
- U4 pad 14: (no net) -> unconnected-(U4-Pad14)
- U4 pad 8: (no net) -> unconnected-(U4D---Pad8)
- U4 pad 9: (no net) -> unconnected-(U4D-+-Pad9)

Commit message: Huella de la tiva, conectores SPI
Parts:
- moved JTIVAR1 227.9 mm to (239.3, 104.1)
- moved JTIVAL1 195.4 mm to (196.1, 104.1)
- moved CDESPOT1 77.4 mm to (127.5, 29.3)
- moved CPOT1 77.4 mm to (127.5, 32.7)
- moved RPOT1 77.4 mm to (127.9, 21.2)
- moved CDES1 44.5 mm to (19.8, 23.5)
- moved D5 44.5 mm to (31.0, 25.0)
- moved J_DC1 44.5 mm to (19.2, 38.0)
- moved R1 44.5 mm to (32.4, 19.1)
- moved RGND0 44.5 mm to (32.3, 34.0)
- moved C1 22.5 mm to (57.5, 31.1)
- moved J1 22.5 mm to (107.5, 17.9)
- moved J2 22.5 mm to (88.3, 33.5)
- moved JA1 22.5 mm to (88.3, 18.0)
- moved JA2 22.5 mm to (93.0, 33.5)
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Changed lines of the file:
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@@
 	(footprint "Connector_PinHeader_2.54mm:PinHeader_1x01_P2.54mm_Vertical"
 		(layer "F.Cu")
-		(at 79.8 18.92)
+		(at 102.3 18)
 		(descr "Through hole straight pin header, 1x01, 2.54mm pitch, single row")
 		(tags "Through hole pin header THT 1x01 2.54mm single row")
@@
 	(footprint "Resistor_SMD:R_1206_3216Metric_Pad1.30x1.75mm_HandSolder"
 		(layer "F.Cu")
-		(at 32.66 63.58)
+		(at 32.43 19.08)
 		(descr "Resistor SMD 1206 (3216 Metric), square (rectangular) end terminal, IPC_7351 nominal with elongated pad for handsoldering. (Body size source: IPC-SM-782 page 72, https://www.pcb-3d.com/wordpress/wp-content/uploads/ipc-sm-782a_amendment_1_and_2.pdf), generated with kicad-footprint-generator")
 		(tags "resistor handsolder")
@@
 	(footprint "TerminalBlock_Phoenix:TerminalBlock_Phoenix_MKDS-1,5-2-5.08_1x02_P5.08mm_Horizontal"
 		(layer "F.Cu")
-		(at 19.42 82.5)
+		(at 19.19 38)
 		(descr "Terminal Block Phoenix MKDS-1,5-2-5.08, 2 pins, pitch 5.08mm, size 10.2x9.8mm, drill diameter 1.3mm, pad diameter 2.6mm, http://www.farnell.com/datasheets/100425.pdf, script-generated using https://gitlab.com/kicad/libraries/kicad-footprint-generator/-/tree/master/scripts/TerminalBlock_Phoenix")
 		(tags "THT Terminal Block Phoenix MKDS-1,5-2-5.08 pitch 5.08mm size 10.2x9.8mm drill 1.3mm pad 2.6mm")
@@
 	(footprint "Resistor_SMD:R_1206_3216Metric_Pad1.30x1.75mm_HandSolder"
 		(layer "F.Cu")
-		(at 32.5 78.5)
+		(at 32.27 34)
 		(descr "Resistor SMD 1206 (3216 Metric), square (rectangular) end terminal, IPC_7351 nominal with elongated pad for handsoldering. (Body size source: IPC-SM-782 page 72, https://www.pcb-3d.com/wordpress/wp-content/uploads/ipc-sm-782a_amendment_1_and_2.pdf), generated with kicad-footprint-generator")
 		(tags "resistor handsolder")
@@
 	(footprint "Connector_PinHeader_2.54mm:PinHeader_1x05_P2.54mm_Vertical"
 		(layer "F.Cu")
-		(at 70.5 18.92)
+		(at 93 18)
 		(descr "Through hole straight pin header, 1x05, 2.54mm pitch, single row")
 		(tags "Through hole pin header THT 1x05 2.54mm single row")
@@
 	(footprint "Connector_PinHeader_2.54mm:PinHeader_1x01_P2.54mm_Vertical"
 		(layer "F.Cu")
-		(at 79.8 28.22)
+		(at 102.3 27.3)
 		(descr "Through hole straight pin header, 1x01, 2.54mm pitch, single row")
 		(tags "Through hole pin header THT 1x01 2.54mm single row")
@@
 	(footprint "Connector_PinHeader_2.54mm:PinHeader_1x04_P2.54mm_Vertical"
 		(layer "F.Cu")
-		(at 70.5 34.42)
+		(at 93 33.5)
 		(descr "Through hole straight pin header, 1x04, 2.54mm pitch, single row")
 		(tags "Through hole pin header THT 1x04 2.54mm single row")
@@
 	(footprint "TerminalBlock_Phoenix:TerminalBlock_Phoenix_MKDS-1,5-3-5.08_1x03_P5.08mm_Horizontal"
 		(layer "F.Cu")
-		(at 65.92 67.5)
+		(at 127.915 21.1725)
 		(descr "Terminal Block Phoenix MKDS-1,5-3-5.08, 3 pins, pitch 5.08mm, size 15.2x9.8mm, drill diameter 1.3mm, pad diameter 2.6mm, http://www.farnell.com/datasheets/100425.pdf, script-generated using https://gitlab.com/kicad/libraries/kicad-footprint-generator/-/tree/master/scripts/TerminalBlock_Phoenix")
 		(tags "THT Terminal Block Phoenix MKDS-1,5-3-5.08 pitch 5.08mm size 15.2x9.8mm drill 1.3mm pad 2.6mm")
@@
 	(footprint "Connector_PinHeader_2.54mm:PinHeader_1x04_P2.54mm_Vertical"
 		(layer "F.Cu")
-		(at 65.85 34.42)
+		(at 88.35 33.5)
 		(descr "Through hole straight pin header, 1x04, 2.54mm pitch, single row")
 		(tags "Through hole pin header THT 1x04 2.54mm single row")
@@
 	(footprint "Capacitor_THT:C_Radial_D12.5mm_H20.0mm_P5.00mm"
 		(layer "F.Cu")
-		(at 20 68)
+		(at 19.77 23.5)
 		(descr "C, Radial series, Radial, pin pitch=5.00mm, diameter=12.5mm, height=20mm, Non-Polar Electrolytic Capacitor")
 		(tags "C Radial series Radial pin pitch 5.00mm diameter 12.5mm height 20mm Non-Polar Electrolytic Capacitor")
@@
 	(footprint "Connector_PinHeader_2.54mm:PinHeader_1x01_P2.54mm_Vertical"
 		(layer "F.Cu")
-		(at 79.8 23.57)
+		(at 102.3 22.65)
 		(descr "Through hole straight pin header, 1x01, 2.54mm pitch, single row")
 		(tags "Through hole pin header THT 1x01 2.54mm single row")
@@
 	(footprint "Capacitor_SMD:C_1206_3216Metric_Pad1.33x1.80mm_HandSolder"
 		(layer "F.Cu")
-		(at 35 32 -90)
+		(at 57.5 31.08 -90)
 		(descr "Capacitor SMD 1206 (3216 Metric), square (rectangular) end terminal, IPC_7351 nominal with elongated pad for handsoldering. (Body size source: IPC-SM-782 page 76, https://www.pcb-3d.com/wordpress/wp-content/uploads/ipc-sm-782a_amendment_1_and_2.pdf), generated with kicad-footprint-generator")
 		(tags "capacitor handsolder")
@@
 	(footprint "Capacitor_SMD:C_1206_3216Metric_Pad1.33x1.80mm_HandSolder"
 		(layer "F.Cu")
-		(at 65.5 79)
+		(at 127.495 32.6725)
 		(descr "Capacitor SMD 1206 (3216 Metric), square (rectangular) end terminal, IPC_7351 nominal with elongated pad for handsoldering. (Body size source: IPC-SM-782 page 76, https://www.pcb-3d.com/wordpress/wp-content/uploads/ipc-sm-782a_amendment_1_and_2.pdf), generated with kicad-footprint-generator")
 		(tags "capacitor handsolder")
@@
 	(footprint "Capacitor_SMD:C_1206_3216Metric_Pad1.33x1.80mm_HandSolder"
 		(layer "F.Cu")
-		(at 65.5 75.65)
+		(at 127.495 29.3225)
 		(descr "Capacitor SMD 1206 (3216 Metric), square (rectangular) end terminal, IPC_7351 nominal with elongated pad for handsoldering. (Body size source: IPC-SM-782 page 76, https://www.pcb-3d.com/wordpress/wp-content/uploads/ipc-sm-782a_amendment_1_and_2.pdf), generated with kicad-footprint-generator")
 		(tags "capacitor handsolder")
@@
 	(footprint "Connector_PinHeader_2.54mm:PinHeader_2x10_P2.54mm_Vertical"
 		(layer "F.Cu")
-		(at 28 18.84)
+		(at 239.3188 104.14)
 		(descr "Through hole straight pin header, 2x10, 2.54mm pitch, double rows")
 		(tags "Through hole pin header THT 2x10 2.54mm double row")
@@
 	(footprint "Connector_PinHeader_2.54mm:PinHeader_2x10_P2.54mm_Vertical"
 		(layer "F.Cu")
-		(at 20.34 18.92)
+		(at 196.1388 104.14)
 		(descr "Through hole straight pin header, 2x10, 2.54mm pitch, double rows")
 		(tags "Through hole pin header THT 2x10 2.54mm double row")
@@
 	(footprint "Connector_PinHeader_2.54mm:PinHeader_1x05_P2.54mm_Vertical"
 		(layer "F.Cu")
-		(at 65.85 18.92)
+		(at 88.35 18)
 		(descr "Through hole straight pin header, 1x05, 2.54mm pitch, single row")
 		(tags "Through hole pin header THT 1x05 2.54mm single row")
@@
 	(footprint "TerminalBlock_Phoenix:TerminalBlock_Phoenix_MKDS-1,5-3-5.08_1x03_P5.08mm_Horizontal"
 		(layer "F.Cu")
-		(at 36.415 22.6725)
+		(at 58.915 21.7525)
 		(descr "Terminal Block Phoenix MKDS-1,5-3-5.08, 3 pins, pitch 5.08mm, size 15.2x9.8mm, drill diameter 1.3mm, pad diameter 2.6mm, http://www.farnell.com/datasheets/100425.pdf, script-generated using https://gitlab.com/kicad/libraries/kicad-footprint-generator/-/tree/master/scripts/TerminalBlock_Phoenix")
 		(tags "THT Terminal Block Phoenix MKDS-1,5-3-5.08 pitch 5.08mm size 15.2x9.8mm drill 1.3mm pad 2.6mm")
@@
 	(footprint "Connector_PinHeader_2.54mm:PinHeader_1x04_P2.54mm_Vertical"
 		(layer "F.Cu")
-		(at 79.8 34.42)
+		(at 102.3 33.5)
 		(descr "Through hole straight pin header, 1x04, 2.54mm pitch, single row")
 		(tags "Through hole pin header THT 1x04 2.54mm single row")
@@
 	(footprint "Connector_PinHeader_2.54mm:PinHeader_1x06_P2.54mm_Vertical"
 		(layer "F.Cu")
-		(at 85 18.84)
+		(at 107.5 17.92)
 		(descr "Through hole straight pin header, 1x06, 2.54mm pitch, single row")
 		(tags "Through hole pin header THT 1x06 2.54mm single row")
@@
 	(footprint "Connector_PinHeader_2.54mm:PinHeader_1x05_P2.54mm_Vertical"
 		(layer "F.Cu")
-		(at 75.15 18.92)
+		(at 97.65 18)
 		(descr "Through hole straight pin header, 1x05, 2.54mm pitch, single row")
 		(tags "Through hole pin header THT 1x05 2.54mm single row")
@@
 	(footprint "Connector_PinHeader_2.54mm:PinHeader_1x04_P2.54mm_Vertical"
 		(layer "F.Cu")
-		(at 75.15 34.42)
+		(at 97.65 33.5)
 		(descr "Through hole straight pin header, 1x04, 2.54mm pitch, single row")
 		(tags "Through hole pin header THT 1x04 2.54mm single row")
@@
 	(footprint "LED_THT:LED_D3.0mm"
 		(layer "F.Cu")
-		(at 31.23 69.5)
+		(at 31 25)
 		(descr "LED, diameter 3.0mm, 2 pins, generated by kicad-footprint-generator")
 		(tags "LED")
@@
 	)
 	(gr_line
-		(start 240 50)
-		(end 240 140)
+		(start 193.5988 139.7)
+		(end 193.5988 76.2)
+		(stroke
+			(width 0.1)
+			(type default)
+		)
+		(layer "Dwgs.User")
+	)
+	(gr_line
+		(start 244.3988 139.7)
+		(end 193.5988 139.7)
+		(stroke
+			(width 0.1)
+			(type default)
+		)
+		(layer "Dwgs.User")
+	)
+	(gr_line
+		(start 244.3988 76.2)
+		(end 244.3988 139.7)
+		(stroke
+			(width 0.1)
+			(type default)
+		)
+		(layer "Dwgs.User")
+	)
+	(gr_line
+		(start 193.5988 76.2)
+		(end 244.3988 76.2)
+		(stroke
+			(width 0.1)
+			(type default)
+		)
+		(layer "Dwgs.User")
+	)
+	(gr_line
+		(start 254 41.36)
+		(end 254 131.36)
 		(stroke
 			(width 0.05)
@@
 	)
 	(gr_line
-		(start 170 50)
-		(end 240 50)
+		(start 184 41.36)
+		(end 254 41.36)
 		(stroke
 			(width 0.05)
@@
 	)
 	(gr_line
-		(start 170 140)
-		(end 170 50)
+		(start 184 131.36)
+		(end 184 41.36)
 		(stroke
 			(width 0.05)
@@
 	)
 	(gr_line
-		(start 240 140)
-		(end 170 140)
+		(start 254 131.36)
+		(end 184 131.36)
 		(stroke
 			(width 0.05)
@@
 		(layer "Edge.Cuts")
 	)
+	(group ""
+		(members "90a4f889-66e9-4b68-8fa0-f3c773b6f2c6" "97a83688-62e3-450e-9d91-495bcda43466")
+	)
+	(group ""
+		(members "18033340-b943-40df-b94e-f7dd02137384" "69023ede-4c98-4fe2-bd8f-8d5988825f4a"
+			"6f78117f-1b06-4491-8ae4-bf35389e7e8b" "a0f84381-85ee-4dc9-9669-f04f50e49eca"
+			"e9c107d0-875e-4116-88bf-3cb33b7b66ec"
+		)
+	)
+	(group ""
+		(members "42953bd3-bd4c-4167-abe9-684f56a67b1f" "499c7059-cf3d-48c4-9718-59191329168a"
+			"81717b9b-7a9a-462d-80a5-f58240868900" "d719915f-fe55-4999-aaae-feb683d98be7"
+			"f430abb7-9baf-4bc8-8099-57171e1e2254"
+		)
+	)
 	(embedded_fonts no)

Commit message: Colocacion de mosfets y drivers
Parts:
- removed QAH1, QAL1, QBH1, QBL1, QCH1, QCL1: IRLR2905TRPBF, Package_TO_SOT_THT:TO-5-3
- removed U1, U2, U3: ~, Package_DIP:CERDIP-8_W7.62mm_SideBrazed_LongPads_Socket
- added MOSFET1: IRFR1205TRPBF, IRFR1205TRPBF:D-PAK_TO-252AA_INF, B.Cu at (218.8, 49.8)
- added MOSFET2: IRFR1205TRPBF, IRFR1205TRPBF:D-PAK_TO-252AA_INF, F.Cu at (218.8, 49.8)
- added MOSFET3: IRFR1205TRPBF, IRFR1205TRPBF:D-PAK_TO-252AA_INF, B.Cu at (231.0, 49.8)
- added MOSFET4: IRFR1205TRPBF, IRFR1205TRPBF:D-PAK_TO-252AA_INF, F.Cu at (231.0, 49.8)
- added MOSFET5: IRFR1205TRPBF, IRFR1205TRPBF:D-PAK_TO-252AA_INF, B.Cu at (206.6, 49.8)
- added MOSFET6: IRFR1205TRPBF, IRFR1205TRPBF:D-PAK_TO-252AA_INF, F.Cu at (206.6, 49.8)
- added REF**: MountingHole_3.2mm_M3, MountingHole:MountingHole_3.2mm_M3, F.Cu at (243.5, 123.5)
- added REF**: MountingHole_3.2mm_M3, MountingHole:MountingHole_3.2mm_M3, F.Cu at (182.5, 42.5)
- added REF**: MountingHole_3.2mm_M3, MountingHole:MountingHole_3.2mm_M3, F.Cu at (243.5, 42.5)
- added REF**: MountingHole_3.2mm_M3, MountingHole:MountingHole_3.2mm_M3, F.Cu at (182.5, 123.5)
- added U10: IR2301SPBF, Package_SO:SOIC-8_3.9x4.9mm_P1.27mm, F.Cu at (218.8, 63.0)
- added U11: IR2301SPBF, Package_SO:SOIC-8_3.9x4.9mm_P1.27mm, F.Cu at (231.0, 63.0)
- added U9: IR2301SPBF, Package_SO:SOIC-8_3.9x4.9mm_P1.27mm, F.Cu at (207.5, 63.1)
- moved D3 259.0 mm to (300.8, 82.0), turned to 180 degrees
- moved CCDES1 258.6 mm to (316.0, 116.5)
- moved CADES1 256.9 mm to (265.5, 113.0)
- moved CABO1 256.9 mm to (266.2, 83.1)
- moved CADR1 256.9 mm to (266.2, 86.5)
- moved CAHI1 256.9 mm to (266.2, 89.8)
- moved CALI1 256.9 mm to (266.2, 93.2)
- moved D2 256.9 mm to (271.4, 82.5)
- moved RAHI1 256.9 mm to (266.2, 103.2)
- moved RALI1 256.9 mm to (266.2, 106.5)
- moved RGAH1 256.9 mm to (266.2, 96.7)
- moved RGAL1 256.9 mm to (266.2, 100.0)
- moved CBBO1 256.5 mm to (289.8, 90.2)
- moved CBDES1 256.5 mm to (289.3, 113.5)
- moved CBDR1 256.5 mm to (289.8, 93.5)
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Connections:
- JC1 pad 5: unconnected-(JC1-Pin_5-Pad5) -> GNDPWR
- JTIVAL1 pad 13: unconnected-(JTIVAL1-Pin_13-Pad13) -> SCLK

Commit message: Colocacion de dispositivos de potencia
Parts:
- added JSPI1: Conn_01x07_Pin, Connector_PinHeader_2.54mm:PinHeader_1x07_P2.54mm_Vertical, F.Cu at (181.4, 100.8)
- moved J_DC1 192.0 mm to (211.1, 44.0), turned to 180 degrees
- moved CDES1 175.9 mm to (194.0, 47.5), turned to 90 degrees
- moved JBLDC1 175.0 mm to (232.5, 44.0), turned to 180 degrees
- moved D5 167.9 mm to (196.2, 55.0)
- moved RGND0 167.5 mm to (198.7, 15.1)
- moved C1 164.6 mm to (20.5, 191.4)
- moved R1 164.1 mm to (192.5, 55.0), turned to 90 degrees
- moved CCDES1 104.2 mm to (232.0, 54.9)
- moved CBDES1 90.8 mm to (219.9, 54.9)
- moved D4 82.3 mm to (237.8, 77.2), turned to 90 degrees
- moved CADES1 82.1 mm to (207.4, 54.9)
- moved D3 75.2 mm to (225.8, 77.2), turned to 90 degrees
- moved D2 58.0 mm to (213.7, 77.2), turned to 90 degrees
- moved CABO1 41.8 mm to (263.0, 41.4)
- moved CBDR1 41.8 mm to (286.6, 51.8)
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Connections:
- JTIVAL1 pad 14: unconnected-(JTIVAL1-Pin_14-Pad14) -> CS
- JTIVAL1 pad 15: unconnected-(JTIVAL1-Pin_15-Pad15) -> MISO
- JTIVAL1 pad 16: unconnected-(JTIVAL1-Pin_16-Pad16) -> MOSI

Commit message: Mas colocación de componentes
Parts:
- moved J1 170.1 mm to (268.1, 73.8)
- moved JB3 170.1 mm to (262.9, 89.3)
- moved JBootA1 170.1 mm to (262.9, 73.8)
- moved JBootC1 170.1 mm to (262.9, 83.1)
- moved J2 170.1 mm to (249.0, 89.3)
- moved JB1 170.1 mm to (253.7, 73.8)
- moved JB2 170.1 mm to (258.3, 89.3)
- moved JC1 170.1 mm to (258.3, 73.8)
- moved JBootB1 170.1 mm to (262.9, 78.5)
- moved JA1 154.9 mm to (240.0, 49.7)
- moved DBUCK1 152.4 mm to (190.5, 60.5), turned to -90 degrees
- moved JA2 152.4 mm to (244.5, 49.7)
- moved RdivAH1 151.3 mm to (270.5, 117.6)
- moved RdivAL1 151.3 mm to (270.5, 120.9)
- moved RdivBH1 151.3 mm to (270.5, 94.2)
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
Commit message: Mas colocacion: Testpoints y alguna cosa mas
Parts:
- removed the JA1 at (240.0, 49.7)
- removed the JB1 at (253.7, 73.8)
- removed the JC1 at (258.3, 73.8)
- added JCONTROL1: Conn_01x07_Pin, Connector_PinSocket_2.54mm:PinSocket_1x07_P2.54mm_Vertical, F.Cu at (228.1, 108.4)
- JTIVAL1, JTIVAR1: value Conn_02x10_Top_Bottom -> Conn_02x10_Odd_Even
- RGND0: moved to B.Cu
- moved RGND0 79.9 mm to (239.5, 83.8), turned to 90 degrees
- moved JBootA1 63.6 mm to (225.3, 22.6)
- moved JBootC1 63.5 mm to (225.2, 32.0)
- moved JBootB1 63.5 mm to (225.2, 27.4)
- moved JBEMF1 35.7 mm to (244.5, 100.5)
- moved JB1 30.2 mm to (244.5, 62.5)
- moved JC1 23.2 mm to (244.5, 75.2)
- moved U4 6.07 mm to (215.3, 99.7)
- moved U6 5.89 mm to (201.7, 88.5)
- moved J2 4.77 mm to (244.5, 87.8)
- moved U7 4.61 mm to (215.5, 88.5)
- moved U8 2.93 mm to (229.2, 88.5)
- moved JA1 0.13 mm to (244.6, 49.6)
- renumbered JA2 to JA1, JB2 to JB1, J1 to JBEMF1, JB3 to JC1
Connections:
- JTIVAL1 pad 10: unconnected-(JTIVAL1-Pin_10-Pad10) -> MISO
- JTIVAL1 pad 11: unconnected-(JTIVAL1-Pin_11-Pad11) -> FASE_C_LIN
- JTIVAL1 pad 12: GND -> MOSI
- JTIVAL1 pad 13: SCLK -> FASE_B_LIN
- JTIVAL1 pad 14: CS -> unconnected-(JTIVAL1-Pin_14-Pad14)
- JTIVAL1 pad 15: MISO -> unconnected-(JTIVAL1-Pin_15-Pad15)
- JTIVAL1 pad 16: MOSI -> unconnected-(JTIVAL1-Pin_16-Pad16)
- JTIVAL1 pad 18: unconnected-(JTIVAL1-Pin_18-Pad18) -> DUTY
- JTIVAL1 pad 19: DUTY -> unconnected-(JTIVAL1-Pin_19-Pad19)
- JTIVAL1 pad 2: FASE_B_HIN -> unconnected-(JTIVAL1-Pin_2-Pad2)
- JTIVAL1 pad 3: unconnected-(JTIVAL1-Pin_3-Pad3) -> FASE_B_HIN
- JTIVAL1 pad 4: unconnected-(JTIVAL1-Pin_4-Pad4) -> GND
- JTIVAL1 pad 5: FASE_C_HIN -> unconnected-(JTIVAL1-Pin_5-Pad5)
- JTIVAL1 pad 6: FASE_C_LIN -> SCLK
- JTIVAL1 pad 7: FASE_B_LIN -> unconnected-(JTIVAL1-Pin_7-Pad7)
- JTIVAL1 pad 8: unconnected-(JTIVAL1-Pin_8-Pad8) -> CS
- JTIVAL1 pad 9: unconnected-(JTIVAL1-Pin_9-Pad9) -> FASE_C_HIN
- JTIVAR1 pad 10: BEMFC -> unconnected-(JTIVAR1-Pin_10-Pad10)
- JTIVAR1 pad 12: unconnected-(JTIVAR1-Pin_12-Pad12) -> FASE_A_HIN
- JTIVAR1 pad 14: unconnected-(JTIVAR1-Pin_14-Pad14) -> FASE_A_LIN
- JTIVAR1 pad 16: FASE_A_HIN -> unconnected-(JTIVAR1-Pin_16-Pad16)
- JTIVAR1 pad 17: FASE_A_LIN -> unconnected-(JTIVAR1-Pin_17-Pad17)
- JTIVAR1 pad 19: unconnected-(JTIVAR1-Pin_19-Pad19) -> BEMFC
- JTIVAR1 pad 2: BEMFB -> unconnected-(JTIVAR1-Pin_2-Pad2)
- JTIVAR1 pad 3: unconnected-(JTIVAR1-Pin_3-Pad3) -> BEMFB
Routing:
- added copper zone on In2.Cu, net GND
- added copper zone on In2.Cu, net GNDPWR
- added copper zone on In1.Cu, net VCC

Commit message: Colocación del puente H A
Parts:
- CABO1, CADR1, CAHI1, CALI1, CBBO1, CBDR1, CCBO1, CCDR1, RAHI1, RALI1, RGAH1: moved to B.Cu
- moved CCBO1 89.1 mm to (229.2, 75.8), turned to -90 degrees
- moved CCDR1 83.7 mm to (229.2, 55.0), turned to 180 degrees
- moved CBBO1 76.3 mm to (215.4, 75.8), turned to -90 degrees
- moved CAHI1 75.0 mm to (194.5, 78.5)
- moved CALI1 74.8 mm to (194.5, 81.5), turned to 180 degrees
- moved CBDR1 71.1 mm to (215.5, 55.0), turned to 180 degrees
- moved CABO1 71.0 mm to (200.1, 74.4), turned to 180 degrees
- moved RAHI1 68.0 mm to (199.2, 84.9), turned to -90 degrees
- moved RALI1 62.5 mm to (203.9, 84.9), turned to -90 degrees
- moved CADR1 62.3 mm to (201.5, 55.0), turned to 180 degrees
- moved RGAL1 59.9 mm to (207.7, 81.3), turned to 90 degrees
- moved RGAH1 59.0 mm to (207.8, 75.8), turned to -90 degrees
- moved CBLI1 35.9 mm to (253.7, 59.5)
- moved RBHI1 35.9 mm to (253.7, 76.0)
- moved RGBH1 35.9 mm to (253.7, 69.2)
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Routing:
- net FASE_A: track 0.00 -> 21.4 mm, vias 0 -> 2
- net GAL: track 0.00 -> 18.4 mm, vias 0 -> 2
- net DFALIN: track 0.00 -> 11.6 mm, vias 0 -> 2
- net DFAHIN: track 0.00 -> 10.2 mm, vias 0 -> 1
- net GAH: track 0.00 -> 6.40 mm
- net GNDPWR: track 0.00 -> 4.87 mm, vias 0 -> 9
- net Net-(U9-LO): track 0.00 -> 4.77 mm
- net Net-(U9-HO): track 0.00 -> 4.14 mm, vias 0 -> 1
- net VCC: vias 0 -> 13

Commit message: Colocación final del puente H
Parts:
- CBHI1, CBLI1, CBLI2, CCHI1, RBHI1, RBLI1, RCHI1, RCLI1, RGAL1, RGBH1, RGBL1, RGCH1, RGCL1: moved to B.Cu
- moved CBLI2 72.8 mm to (228.3, 83.0), turned to -90 degrees
- moved CCHI1 71.7 mm to (228.3, 77.5), turned to -90 degrees
- moved RCHI1 66.5 mm to (231.2, 86.0), turned to -90 degrees
- moved RCLI1 61.0 mm to (235.7, 86.1), turned to -90 degrees
- moved RGCL1 59.5 mm to (240.2, 83.6), turned to 90 degrees
- moved RGCH1 57.1 mm to (240.2, 76.2), turned to -90 degrees
- moved CBLI1 47.8 mm to (212.1, 83.0), turned to -90 degrees
- moved CBHI1 47.1 mm to (212.1, 77.7), turned to -90 degrees
- moved JBootA1 42.1 mm to (207.2, 60.3)
- moved RBHI1 39.5 mm to (215.4, 86.0), turned to -90 degrees
- moved RBLI1 34.2 mm to (220.2, 86.0), turned to -90 degrees
- moved JBootB1 33.3 mm to (223.8, 60.6)
- moved JBootC1 31.8 mm to (239.1, 60.6)
- moved RGBL1 31.2 mm to (224.5, 83.5), turned to 90 degrees
- moved RGBH1 29.9 mm to (224.5, 75.9), turned to -90 degrees
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Connections:
- JSPI1 pad 3: MISO -> CS
- JSPI1 pad 5: MOSI -> MISO
- JSPI1 pad 7: CS -> MOSI
Routing:
- net FASE_B: track 0.00 -> 34.6 mm, vias 0 -> 3
- net VBA: track 0.00 -> 32.9 mm, vias 0 -> 1
- net VBB: track 0.00 -> 32.5 mm, vias 0 -> 1
- net VBC: track 0.00 -> 31.6 mm, vias 0 -> 1
- net GCL: track 0.00 -> 25.6 mm, vias 0 -> 1
- net GNDPWR: track 4.87 -> 29.5 mm, vias 9 -> 17
- net FASE_C: track 0.00 -> 23.1 mm, vias 0 -> 2
- net GBL: track 0.00 -> 22.9 mm, vias 0 -> 1
- net FASE_A: track 21.4 -> 36.9 mm, vias 2 -> 3
- net GND: track 0.00 -> 14.4 mm, vias 0 -> 2
- net DFBHIN: track 0.00 -> 13.8 mm, vias 0 -> 1
- net DFCHIN: track 0.00 -> 13.2 mm, vias 0 -> 1
- net DFBLIN: track 0.00 -> 12.9 mm, vias 0 -> 1
- net DFCLIN: track 0.00 -> 12.6 mm, vias 0 -> 1
- net VCC: track 0.00 -> 10.5 mm, vias 13 -> 2
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