File: ESC_BLDC.kicad_pcb (KiCad board)
At the start: 4 copper layers, 70 x 90 mm, 98 parts, among them J2 Conn_01x04_Pin, U10 IR2301SPBF, U11 IR2301SPBF, U4 LM339, U5 AP1509-50SG-13, U6 MCP6002-xP, U7 MCP6002-xP, U8 MCP6002-xP, U9 IR2301SPBF

Commit message: routing no completo
Parts:
- removed JB1, JC1: Conn_01x04_Pin, Connector_PinHeader_2.54mm:PinHeader_1x04_P2.54mm_Vertical
- added JGA1: Conn_01x03_Pin, Connector_PinHeader_2.54mm:PinHeader_1x03_P2.54mm_Vertical, F.Cu at (189.4, 79.4)
- added JGB1: Conn_01x03_Pin, Connector_PinHeader_2.54mm:PinHeader_1x03_P2.54mm_Vertical, F.Cu at (189.5, 90.3)
- added JGC1: Conn_01x03_Pin, Connector_PinHeader_2.54mm:PinHeader_1x03_P2.54mm_Vertical, F.Cu at (237.8, 95.2)
- RN2, RN3: moved to B.Cu
- moved C1 159.0 mm to (155.3, 107.1), turned to 0 degrees
- moved RdivCH1 131.1 mm to (141.2, 82.0)
- moved RdivCL1 131.0 mm to (141.2, 85.9)
- moved CdesB1 122.9 mm to (155.4, 103.7)
- moved CDESBEMF2 122.6 mm to (155.4, 99.0)
- moved CBYPASS2 122.4 mm to (155.5, 94.2), turned to 180 degrees
- moved Rpullup2 122.0 mm to (149.3, 103.7)
- moved RdivBH1 116.9 mm to (154.8, 81.9)
- moved RdivBL1 116.7 mm to (154.9, 85.9)
- moved CBYPASS1 104.6 mm to (174.0, 104.2)
- moved CdesA1 104.5 mm to (174.1, 99.7)
- moved CBYPASS3 104.3 mm to (174.2, 111.2)
- moved CDESBEMF1 104.0 mm to (174.1, 95.4)
- moved Rpullup3 103.9 mm to (167.7, 120.4)
- moved CDESBEMF3 103.9 mm to (174.2, 115.4)
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Connections:
- JA1 pad 1: FASE_A -> FASE_C
- JA1 pad 2: GAH -> FASE_B
- JA1 pad 3: GAL -> FASE_A
- JBLDC1 pad 1: FASE_A -> FASE_C
- JBLDC1 pad 3: FASE_C -> FASE_A
Routing:
- net FASE_A: track 36.9 -> 103.3 mm, vias 3 -> 4
- net Net-(RN1-Pad2): track 0.00 -> 55.6 mm, vias 0 -> 1
- net GBH: track 6.74 -> 58.6 mm, vias 0 -> 1
- net GAH: track 6.08 -> 47.3 mm, vias 0 -> 1
- net FASE_B: track 34.6 -> 75.6 mm, vias 3 -> 4
- net +3.3V: track 5.61 -> 44.7 mm, vias 0 -> 2
- net GBL: track 22.9 -> 61.1 mm
- net GCH: track 6.89 -> 40.2 mm
- net FASE_C: track 23.1 -> 55.0 mm, vias 2 -> 3
- net GNDPWR: track 29.5 -> 59.3 mm, vias 17 -> 21
- net GAL: track 22.4 -> 47.5 mm
- net Net-(DBUCK1-K): track 0.00 -> 14.9 mm, vias 0 -> 2
- net GCL: track 25.6 -> 35.3 mm
- net NEUTRO: track 0.00 -> 9.55 mm
- net GND: track 14.4 -> 21.3 mm, vias 2 -> 7
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
Commit message: routing analogico
Parts:
- CINVCC1, CINVDD1: footprint Capacitor_SMD:C_Elec_6.3x5.8 -> Capacitor_SMD:C_1206_3216Metric_Pad1.33x1.80mm_HandSolder
- JTIVAL1, JTIVAR1: moved to B.Cu
- moved RdivCH1 103.3 mm to (241.5, 57.5), turned to 180 degrees
- moved RdivAL1 86.7 mm to (172.1, 86.1)
- moved RdivBH1 63.2 mm to (210.4, 51.9)
- moved RdivAH1 61.3 mm to (194.4, 66.5)
- moved JSPI1 11.6 mm to (186.0, 103.3)
- moved CINVCC1 4.79 mm to (188.2, 68.8), turned to 180 degrees
- moved CINVDD1 2.68 mm to (182.4, 68.8), turned to 180 degrees
- moved JTIVAL1 2.54 mm to (192.7, 100.8), turned to 180 degrees
- moved JTIVAR1 2.54 mm to (235.9, 100.8), turned to 180 degrees
- moved RN2 1.83 mm to (245.2, 53.5)
- moved JGC1 1.51 mm to (236.3, 95.2)
- moved RN3 1.07 mm to (241.5, 54.7)
- moved RN1 0.85 mm to (245.2, 55.7)
Routing:
- net Net-(U7A-+): track 0.00 -> 98.0 mm, vias 0 -> 2
- net Net-(U8A-+): track 0.00 -> 92.1 mm, vias 0 -> 2
- net FASE_C_LIN: track 0.00 -> 75.2 mm
- net FASE_C_HIN: track 0.00 -> 70.8 mm
- net FASE_B_LIN: track 0.00 -> 68.9 mm
- net FASE_B_HIN: track 0.00 -> 68.1 mm, vias 0 -> 1
- net FASE_A_HIN: track 0.00 -> 59.8 mm, vias 0 -> 1
- net FASE_A_LIN: track 0.00 -> 58.4 mm, vias 0 -> 3
- net Net-(U6A-+): track 0.00 -> 54.3 mm, vias 0 -> 2
- net FASE_B: track 75.6 -> 98.2 mm
- net FASE_C: track 55.0 -> 68.1 mm, vias 3 -> 4
- net +3.3V: track 44.7 -> 38.3 mm
- net Net-(RN1-Pad2): track 55.6 -> 50.3 mm, vias 1 -> 0
- net GND: track 21.3 -> 17.2 mm
- net FASE_A: track 103.3 -> 107.0 mm
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
Commit message: Mal routing
Parts:
- removed J2: Conn_01x04_Pin, Connector_PinHeader_2.54mm:PinHeader_1x04_P2.54mm_Vertical
- removed JBEMF1: Conn_01x06_Pin, Connector_PinHeader_2.54mm:PinHeader_1x06_P2.54mm_Vertical
- CBYPASS1, CBYPASS2, CBYPASS3, CDESBEMF2, CdesA1, CdesB1, CdesC1, RdivAL1, RdivBL1, RdivCL1, Rpullup1, Rpullup2, Rpullup3: moved to B.Cu
- moved RdivCL1 103.3 mm to (243.4, 101.2)
- moved Rpullup2 65.9 mm to (214.9, 97.8)
- moved CdesB1 65.6 mm to (219.6, 90.2)
- moved CBYPASS2 60.1 mm to (214.0, 107.8), turned to 90 degrees
- moved RdivBL1 59.0 mm to (213.6, 92.2), turned to -90 degrees
- moved Rpullup3 58.9 mm to (223.6, 101.8)
- moved CDESBEMF2 58.0 mm to (213.4, 102.0), turned to 180 degrees
- moved CDESBEMF3 54.3 mm to (226.8, 102.0)
- moved Rpullup1 51.5 mm to (219.8, 103.2), turned to -90 degrees
- moved C1 42.2 mm to (197.0, 100.8)
- moved CDESBEMF1 39.8 mm to (213.4, 102.0), turned to 180 degrees
- moved CBYPASS1 34.6 mm to (207.8, 96.8)
- moved CdesC1 34.4 mm to (206.2, 107.4), turned to -90 degrees
- moved CBYPASS3 33.4 mm to (206.0, 100.8)
- moved RdivAL1 29.4 mm to (200.8, 92.2)
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Routing:
- net +3.3V: track 38.3 -> 102.3 mm, vias 2 -> 6
- net BEMFC: track 0.00 -> 46.2 mm, vias 0 -> 2
- net BEMFB: track 0.00 -> 33.6 mm, vias 0 -> 1
- net BEMFA: track 0.00 -> 32.9 mm, vias 0 -> 1
- net NEUTRO: track 9.55 -> 40.2 mm, vias 0 -> 3
- net Net-(U4C--): track 0.00 -> 28.6 mm, vias 0 -> 2
- net Net-(U4B--): track 0.00 -> 26.6 mm, vias 0 -> 2
- net DUTY: track 5.95 -> 30.8 mm
- net GND: track 17.2 -> 32.6 mm, vias 7 -> 15
- net Net-(U8A-+): track 92.1 -> 100.9 mm, vias 2 -> 3
- net Net-(U7A-+): track 98.0 -> 105.5 mm, vias 2 -> 4
- net Net-(U4A-+): track 0.00 -> 7.30 mm, vias 0 -> 1
- net FASE_C3.3V: track 0.00 -> 6.15 mm, vias 0 -> 1
- net FASE_A3.3V: track 0.00 -> 5.63 mm, vias 0 -> 1
- net Net-(U6A-+): track 54.3 -> 58.5 mm
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