File: ESC_BLDC.kicad_sch (KiCad schematic)
At the start: 94 parts, among them J2 Conn_01x04_Pin, U10 IR2301SPBF, U11 IR2301SPBF, U4 LM339, U5 AP1509-50SG-13, U6 MCP6002-xP, U7 MCP6002-xP, U8 MCP6002-xP, U9 IR2301SPBF

Commit message: Colocación del puente H A
Connections:
- net VBA: no longer CABO1.2, D2.1 (K)
- new net: CABO1.2, D2.1 (K)
Changed lines of the file:
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@@
 	)
 	(junction
-		(at 69.85 29.21)
-		(diameter 0)
-		(color 0 0 0 0)
-	)
-	(junction
 		(at 82.55 102.87)
 		(diameter 0)
@@
 	(wire
 		(pts
+			(xy 66.04 38.1) (xy 69.85 38.1)
+		)
+		(stroke
+			(width 0)
+			(type default)
+		)
+	)
+	(wire
+		(pts
 			(xy 280.67 39.37) (xy 279.4 39.37)
 		)
@@
 		)
 	)
-	(wire
-		(pts
-			(xy 69.85 38.1) (xy 66.04 38.1)
-		)
-		(stroke
-			(width 0)
-			(type default)
-		)
-	)
 	(polyline
 		(pts
@@
 	(wire
 		(pts
-			(xy 69.85 29.21) (xy 69.85 38.1)
-		)
-		(stroke
-			(width 0)
-			(type default)
-		)
-	)
-	(wire
-		(pts
 			(xy 48.26 29.21) (xy 48.26 38.1)
 		)
@@
 	(wire
 		(pts
-			(xy 68.58 29.21) (xy 69.85 29.21)
+			(xy 68.58 29.21) (xy 73.66 29.21)
 		)
 		(stroke
@@
 	(wire
 		(pts
-			(xy 69.85 29.21) (xy 73.66 29.21)
-		)
-		(stroke
-			(width 0)
-			(type default)
-		)
-	)
-	(wire
-		(pts
 			(xy 201.93 222.25) (xy 217.17 222.25)
 		)
@@
 	(wire
 		(pts
-			(xy 69.85 26.67) (xy 69.85 29.21)
-		)
-		(stroke
-			(width 0)
-			(type default)
-		)
-	)
-	(wire
-		(pts
 			(xy 48.26 29.21) (xy 60.96 29.21)
 		)
@@
 	(wire
 		(pts
+			(xy 69.85 26.67) (xy 69.85 38.1)
+		)
+		(stroke
+			(width 0)
+			(type default)
+		)
+	)
+	(wire
+		(pts
 			(xy 81.28 151.13) (xy 85.09 151.13)
 		)
@@
 		(length 0.6)
 		(shape dot)
-		(at 40.64 45.72 0)
+		(at 69.85 102.87 0)
 		(fields_autoplaced yes)
 		(effects
@@
 		)
 		(property "Netclass" "Potencia"
-			(at 41.3385 45.12 0)
+			(at 70.5485 102.27 0)
 			(effects
 				(font
@@
 		)
 		(property "Component Class" ""
-			(at -179.07 11.43 0)
+			(at -149.86 68.58 0)
 			(effects
 				(font
@@
 		(length 0.6)
 		(shape dot)
-		(at 69.85 102.87 0)
+		(at 213.36 45.72 0)
 		(fields_autoplaced yes)
 		(effects
 			(font
 				(size 1.27 1.27)
-				(color 189 16 38 1)
+				(color 0 39 189 1)
 			)
 			(justify left bottom)
 		)
-		(property "Netclass" "Potencia"
-			(at 70.5485 102.27 0)
+		(property "Netclass" "Digital"
+			(at 214.0585 45.12 0)
 			(effects
 				(font
@@
 		)
 		(property "Component Class" ""
-			(at -149.86 68.58 0)
+			(at -6.35 11.43 0)
 			(effects
 				(font
@@
 		(length 0.6)
 		(shape dot)
-		(at 213.36 45.72 0)
+		(at 85.09 91.44 0)
 		(fields_autoplaced yes)
 		(effects
 			(font
 				(size 1.27 1.27)
-				(color 0 39 189 1)
+				(color 189 16 38 1)
 			)
 			(justify left bottom)
 		)
-		(property "Netclass" "Digital"
-			(at 214.0585 45.12 0)
+		(property "Netclass" "Potencia"
+			(at 85.7885 90.84 0)
 			(effects
 				(font
@@
 		)
 		(property "Component Class" ""
-			(at -6.35 11.43 0)
+			(at -134.62 57.15 0)
 			(effects
 				(font
@@
 		(length 0.6)
 		(shape dot)
-		(at 85.09 91.44 0)
+		(at 210.82 248.92 0)
 		(fields_autoplaced yes)
 		(effects
@@
 		)
 		(property "Netclass" "Potencia"
-			(at 85.7885 90.84 0)
+			(at 211.5185 248.32 0)
 			(effects
 				(font
@@
 		)
 		(property "Component Class" ""
-			(at -134.62 57.15 0)
+			(at -8.89 214.63 0)
 			(effects
 				(font
@@
 		(length 0.6)
 		(shape dot)
-		(at 210.82 248.92 0)
+		(at 68.58 115.57 0)
 		(fields_autoplaced yes)
 		(effects
@@
 		)
 		(property "Netclass" "Potencia"
-			(at 211.5185 248.32 0)
+			(at 69.2785 114.97 0)
 			(effects
 				(font
@@
 		)
 		(property "Component Class" ""
-			(at -8.89 214.63 0)
+			(at -151.13 81.28 0)
 			(effects
 				(font
@@
 		(length 0.6)
 		(shape dot)
-		(at 68.58 115.57 0)
+		(at 30.48 52.07 0)
 		(fields_autoplaced yes)
 		(effects
 			(font
 				(size 1.27 1.27)
-				(color 189 16 38 1)
+				(color 0 39 189 1)
 			)
 			(justify left bottom)
 		)
-		(property "Netclass" "Potencia"
-			(at 69.2785 114.97 0)
+		(property "Netclass" "Digital"
+			(at 31.1785 51.47 0)
 			(effects
 				(font
@@
 		)
 		(property "Component Class" ""
-			(at -151.13 81.28 0)
+			(at -189.23 17.78 0)
 			(effects
 				(font
@@
 		(length 0.6)
 		(shape dot)
-		(at 30.48 52.07 0)
+		(at 166.37 100.33 0)
 		(fields_autoplaced yes)
 		(effects
 			(font
 				(size 1.27 1.27)
-				(color 0 39 189 1)
+				(color 24 189 0 1)
 			)
 			(justify left bottom)
 		)
-		(property "Netclass" "Digital"
-			(at 31.1785 51.47 0)
+		(property "Netclass" "Analogico"
+			(at 167.0685 99.73 0)
 			(effects
 				(font
@@
 		)
 		(property "Component Class" ""
-			(at -189.23 17.78 0)
+			(at -53.34 66.04 0)
 			(effects
 				(font
@@
 		(length 0.6)
 		(shape dot)
-		(at 166.37 100.33 0)
+		(at 68.58 38.1 0)
 		(fields_autoplaced yes)
 		(effects
@@
 		)
 		(property "Netclass" "Analogico"
-			(at 167.0685 99.73 0)
+			(at 69.2785 37.5 0)
 			(effects
 				(font
@@
 		)
 		(property "Component Class" ""
-			(at -53.34 66.04 0)
+			(at -151.13 3.81 0)
 			(effects
 				(font
@@
 		(length 0.6)
 		(shape dot)
-		(at 165.1 217.17 0)
+		(at 44.45 40.64 0)
 		(fields_autoplaced yes)
 		(effects
 			(font
 				(size 1.27 1.27)
-				(color 24 189 0 1)
+				(color 0 39 189 1)
 			)
 			(justify left bottom)
 		)
-		(property "Netclass" "Analogico"
-			(at 165.7985 216.57 0)
+		(property "Netclass" "Digital"
+			(at 45.1485 40.04 0)
 			(effects
 				(font
@@
 		)
 		(property "Component Class" ""
-			(at -54.61 182.88 0)
+			(at -175.26 6.35 0)
 			(effects
 				(font
@@
 		(length 0.6)
 		(shape dot)
-		(at 40.64 48.26 0)
+		(at 165.1 217.17 0)
 		(fields_autoplaced yes)
 		(effects
 			(font
 				(size 1.27 1.27)
-				(color 189 16 38 1)
+				(color 24 189 0 1)
 			)
 			(justify left bottom)
 		)
-		(property "Netclass" "Potencia"
-			(at 41.3385 47.66 0)
+		(property "Netclass" "Analogico"
+			(at 165.7985 216.57 0)
 			(effects
 				(font
@@
 		)
 		(property "Component Class" ""
-			(at -179.07 13.97 0)
+			(at -54.61 182.88 0)
 			(effects
 				(font
@@
 		(length 0.6)
 		(shape dot)
-		(at 71.755 29.21 0)
-		(fields_autoplaced yes)
-		(effects
-			(font
-				(size 1.27 1.27)
-				(color 189 16 38 1)
-			)
-			(justify left bottom)
-		)
-		(property "Netclass" "Potencia"
-			(at 72.4535 28.61 0)
-			(effects
-				(font
-					(size 1.27 1.27)
-				)
-				(justify left)
-				(hide yes)
-			)
-		)
-		(property "Component Class" ""
-			(at -147.955 -5.08 0)
-			(effects
-				(font
-					(size 1.27 1.27)
-					(italic yes)
-				)
-				(hide yes)
-			)
-		)
-	)
-	(netclass_flag ""
-		(length 0.6)
-		(shape dot)
 		(at 85.09 151.13 0)
 		(fields_autoplaced yes)
@@
 		(length 0.6)
 		(shape dot)
+		(at 72.39 29.21 0)
+		(fields_autoplaced yes)
+		(effects
+			(font
+				(size 1.27 1.27)
+				(color 24 189 0 1)
+			)
+			(justify left bottom)
+		)
+		(property "Netclass" "Analogico"
+			(at 73.0885 28.61 0)
+			(effects
+				(font
+					(size 1.27 1.27)
+				)
+				(justify left)
+				(hide yes)
+			)
+		)
+		(property "Component Class" ""
+			(at -147.32 -5.08 0)
+			(effects
+				(font
+					(size 1.27 1.27)
+					(italic yes)
+				)
+				(hide yes)
+			)
+		)
+	)
+	(netclass_flag ""
+		(length 0.6)
+		(shape dot)
 		(at 241.3 163.83 0)
 		(fields_autoplaced yes)
@@
 			(effects
 				(font
+					(size 1.27 1.27)
+					(italic yes)
+				)
+				(hide yes)
+			)
+		)
+	)
+	(netclass_flag ""
+		(length 0.6)
+		(shape dot)
+		(at 44.45 48.26 0)
+		(fields_autoplaced yes)
+		(effects
+			(font
+				(size 1.27 1.27)
+				(color 0 39 189 1)
+			)
+			(justify left bottom)
+		)
+		(property "Netclass" "Digital"
+			(at 45.1485 47.66 0)
+			(effects
+				(font
+					(size 1.27 1.27)
+				)
+				(justify left)
+				(hide yes)
+			)
+		)
+		(property "Component Class" ""
+			(at -175.26 13.97 0)
+			(effects
+				(font

Commit message: Colocación final del puente H
Connections:
- net CS: now also JSPI1.3 (Pin_3); no longer JSPI1.7 (Pin_7)
- net MISO: now also JSPI1.5 (Pin_5); no longer JSPI1.3 (Pin_3)
- net MOSI: now also JSPI1.7 (Pin_7); no longer JSPI1.5 (Pin_5)
- net VBA: now also CABO1.2, D2.1 (K)

Commit message: routing no completo
Parts:
- removed JB1, JC1: Conn_01x04_Pin, Connector_PinHeader_2.54mm:PinHeader_1x04_P2.54mm_Vertical, symbol Connector:Conn_01x04_Pin
- added JGA1, JGB1, JGC1: Conn_01x03_Pin, Connector_PinHeader_2.54mm:PinHeader_1x03_P2.54mm_Vertical, symbol Connector:Conn_01x03_Pin
Connections:
- net FASE_A: now also JA1.3 (Pin_3), JBLDC1.3 (Pin_3); no longer JA1.1 (Pin_1), JBLDC1.1 (Pin_1)
- net FASE_B: now also JA1.2 (Pin_2)
- net FASE_C: now also JA1.1 (Pin_1), JBLDC1.1 (Pin_1); no longer JBLDC1.3 (Pin_3)
- net GAH: now also JGA1.1 (Pin_1); no longer JA1.2 (Pin_2)
- net GAL: now also JGA1.2 (Pin_2); no longer JA1.3 (Pin_3)
- net GBH: now also JGB1.1 (Pin_1)
- net GBL: now also JGB1.2 (Pin_2)
- net GCH: now also JGC1.2 (Pin_2)
- net GCL: now also JGC1.1 (Pin_1)
- net GNDPWR: now also JGA1.3 (Pin_3), JGB1.3 (Pin_3), JGC1.3 (Pin_3)
Other:
- moved on the sheet: JA1
