File: ESC_BLDC.kicad_sch (KiCad schematic)
At the start: 95 parts, among them J2 Conn_01x04_Pin, U10 IR2301SPBF, U11 IR2301SPBF, U4 LM339, U5 AP1509-50SG-13, U6 MCP6002-xP, U7 MCP6002-xP, U8 MCP6002-xP, U9 IR2301SPBF

Commit message: routing analogico
Parts:
- CINVCC1, CINVDD1: footprint Capacitor_SMD:C_Elec_6.3x5.8 -> Capacitor_SMD:C_1206_3216Metric_Pad1.33x1.80mm_HandSolder
Changed lines of the file:
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@@
 			)
 		)
-		(property "Footprint" "Capacitor_SMD:C_Elec_6.3x5.8"
+		(property "Footprint" "Capacitor_SMD:C_1206_3216Metric_Pad1.33x1.80mm_HandSolder"
 			(at 254.3048 166.37 0)
 			(effects
@@
 			)
 		)
-		(property "Footprint" "Capacitor_SMD:C_Elec_6.3x5.8"
+		(property "Footprint" "Capacitor_SMD:C_1206_3216Metric_Pad1.33x1.80mm_HandSolder"
 			(at 194.0052 172.72 0)
 			(effects
